File: hs2/non-deployables_IXOLAR/non-deployables_XTE-SF.kicad_pcb (KiCad board)
At the start: 2 copper layers, 8 parts

Commit message: setting up prototype arrays
Parts:
- removed SC1, SC2, SC3, SC4, SC5, SC6, SC7, SC8: XTE-SF, solar_cells:xte-sf

Commit message: started prototype pcbs for 2 panel boards
Parts:
- added D1: 1N5400, Diode_THT:D_DO-201AD_P15.24mm_Horizontal, F.Cu at (65.1, 32.5)
- added D2: 1N5400, Diode_THT:D_DO-201AD_P15.24mm_Horizontal, F.Cu at (149.9, 32.5)
- added D3: 1N5400, Diode_THT:D_DO-201AD_P15.24mm_Horizontal, F.Cu at (42.6, 32.5)
- added D4: 1N5400, Diode_THT:D_DO-201AD_P15.24mm_Horizontal, F.Cu at (240.1, 35.0)
- added D5: 1N5400, Diode_THT:D_DO-201AD_P15.24mm_Horizontal, F.Cu at (382.4, 35.0)
- added J1: Conn_01x01_Pin, Connector_Wire:SolderWirePad_1x01_SMD_5x10mm, F.Cu at (95.0, 32.5)
- added J2: Conn_01x01_Pin, Connector_Wire:SolderWirePad_1x01_SMD_5x10mm, F.Cu at (295.0, 35.0)
- added Other_Board1: Conn_01x01_Pin, Connector_Wire:SolderWirePad_1x01_SMD_5x10mm, F.Cu at (195.0, 32.5)
- added Other_Board2: Conn_01x01_Pin, Connector_Wire:SolderWirePad_1x01_SMD_5x10mm, F.Cu at (355.0, 35.0)
- added SC1: Solar_Cell, solar_cells:XOLAR_SM401K08TF, F.Cu at (65.0, 100.0)
- added SC10: Solar_Cell, solar_cells:XOLAR_SM401K08TF, F.Cu at (157.5, 57.5)
- added SC11: Solar_Cell, solar_cells:XOLAR_SM401K08TF, F.Cu at (265.0, 60.0)
- added SC12: Solar_Cell, solar_cells:XOLAR_SM401K08TF, F.Cu at (357.5, 60.0)
- added SC13: Solar_Cell, solar_cells:XOLAR_SM401K08TF, F.Cu at (265.0, 102.5)
- added SC14: Solar_Cell, solar_cells:XOLAR_SM401K08TF, F.Cu at (265.0, 145.0)
- added SC15: Solar_Cell, solar_cells:XOLAR_SM401K08TF, F.Cu at (265.0, 187.5)
- added SC16: Solar_Cell, solar_cells:XOLAR_SM401K08TF, F.Cu at (265.0, 230.0)
- added SC17: Solar_Cell, solar_cells:XOLAR_SM401K08TF, F.Cu at (357.5, 102.5)
- added SC18: Solar_Cell, solar_cells:XOLAR_SM401K08TF, F.Cu at (357.5, 145.0)
- added SC19: Solar_Cell, solar_cells:XOLAR_SM401K08TF, F.Cu at (357.5, 187.5)
- added SC2: Solar_Cell, solar_cells:XOLAR_SM401K08TF, F.Cu at (65.0, 142.5)
- added SC20: Solar_Cell, solar_cells:XOLAR_SM401K08TF, F.Cu at (357.5, 230.0)
- added SC3: Solar_Cell, solar_cells:XOLAR_SM401K08TF, F.Cu at (65.0, 185.0)
- added SC4: Solar_Cell, solar_cells:XOLAR_SM401K08TF, F.Cu at (65.0, 227.5)
- added SC5: Solar_Cell, solar_cells:XOLAR_SM401K08TF, F.Cu at (157.5, 100.0)
- added SC6: Solar_Cell, solar_cells:XOLAR_SM401K08TF, F.Cu at (157.5, 142.5)
- added SC7: Solar_Cell, solar_cells:XOLAR_SM401K08TF, F.Cu at (157.5, 185.0)
- added SC8: Solar_Cell, solar_cells:XOLAR_SM401K08TF, F.Cu at (157.5, 227.5)
- added SC9: Solar_Cell, solar_cells:XOLAR_SM401K08TF, F.Cu at (65.0, 57.5)
- added gnd_connector1: Conn_01x01_Pin, Connector_Wire:SolderWirePad_1x01_SMD_5x10mm, F.Cu at (127.5, 32.5)
- added gnd_connector2: Conn_01x01_Pin, Connector_Wire:SolderWirePad_1x01_SMD_5x10mm, F.Cu at (327.5, 35.0)
Routing:
- net Net-(D4-K): track 0.00 -> 148.5 mm
- net Net-(Other_Board2-Pin_1): track 0.00 -> 135.4 mm
- net Net-(D1-K): track 0.00 -> 115.8 mm
- net Net-(D5-A): track 0.00 -> 103.1 mm
- net Net-(SC7--): track 0.00 -> 87.6 mm
- net Net-(SC6--): track 0.00 -> 87.6 mm
- net Net-(SC5--): track 0.00 -> 87.6 mm
- net Net-(SC3--): track 0.00 -> 87.6 mm
- net Net-(SC2--): track 0.00 -> 87.6 mm
- net Net-(SC19--): track 0.00 -> 87.6 mm
- net Net-(SC18--): track 0.00 -> 87.6 mm
- net Net-(SC17--): track 0.00 -> 87.6 mm
- net Net-(SC15--): track 0.00 -> 87.6 mm
- net Net-(SC14--): track 0.00 -> 87.6 mm
- net Net-(SC13--): track 0.00 -> 87.6 mm
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