File: hs2/non-deployables_IXOLAR/non-deployables_XTE-SF.kicad_pcb (KiCad board)
At the start: 2 copper layers, 31 parts, among them J1 Conn_01x01_Pin, J2 Conn_01x01_Pin

Commit message: finished drafting prototype panels
Parts:
- D1, D2, D3, D4, D5: moved to B.Cu
- moved Other_Board2 88.8 mm to (266.2, 31.2)
- moved D1 18.8 mm to (66.4, 51.2)
- moved D2 18.8 mm to (151.1, 51.2)
- moved D3 18.8 mm to (43.9, 51.2)
- moved J1 18.8 mm to (96.2, 51.2)
- moved Other_Board1 18.8 mm to (196.2, 51.2)
- moved SC1 18.8 mm to (66.2, 118.8)
- moved SC10 18.8 mm to (158.8, 76.2)
- moved SC2 18.8 mm to (66.2, 161.2)
- moved SC3 18.8 mm to (66.2, 203.8)
- moved SC4 18.8 mm to (66.2, 246.2)
- moved SC5 18.8 mm to (158.8, 118.8)
- moved SC6 18.8 mm to (158.8, 161.2)
- moved SC7 18.8 mm to (158.8, 203.8)
- moved SC8 18.8 mm to (158.8, 246.2)
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Routing:
- net Net-(Other_Board2-Pin_1): track 135.4 -> 47.9 mm
- net Net-(D4-K): track 148.5 -> 153.9 mm
- net Net-(D1-K): track 115.8 -> 118.9 mm
- added copper zone on F.Cu, net GND1
- added copper zone on F.Cu, net GND2
Other:
- board outline added: 390 x 252.5 mm

Commit message: having problems with smd connectors
Parts:
- J1, J2: moved to B.Cu
- moved D1 8.84 mm to (75.1, 50.0)
- moved D3 1.77 mm to (45.1, 50.0)
Routing:
- net Net-(D1-K): track 118.9 -> 82.9 mm
- net Net-(D1-A): track 75.7 -> 80.6 mm
- net Net-(D4-K): track 153.9 -> 155.7 mm
- net Net-(D4-A): track 69.6 -> 70.9 mm
- net Net-(D3-A): track 26.1 -> 26.8 mm
- removed copper zone on F.Cu, net GND1
- removed copper zone on F.Cu, net GND2

Commit message: prototype board questionable according to KiCAD :cry:
Routing:
- net Net-(D1-K): track 82.9 -> 116.6 mm
- net Net-(D4-K): track 155.7 -> 154.9 mm
- added copper zone on B.Cu, net GND1
- added copper zone on B.Cu, net GND2
Changed lines of the file:
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@@
 		(tags "Diode DO-201AD series Axial Horizontal pin pitch 15.24mm  length 9.5mm diameter 5.2mm")
 		(property "Reference" "D3"
-			(at 0 0 0)
+			(at 7.62 5 0)
 			(layer "B.SilkS")
 			(effects
@@
 		(tags "MeasurementPoint Square SMDPad 5mmx10mm ")
 		(property "Reference" "J1"
-			(at 0 6 90)
+			(at 0 6 270)
 			(layer "B.SilkS")
 			(effects
@@
 		)
 		(property "Value" "Conn_01x01_Pin"
-			(at 5 0 0)
-			(layer "B.Fab")
-			(effects
-				(font
-					(size 1 1)
-					(thickness 0.15)
-				)
-				(justify mirror)
-			)
-		)
-		(property "Datasheet" "~"
+			(at 0 -6.35 270)
+			(layer "B.Fab")
+			(effects
+				(font
+					(size 1 1)
+					(thickness 0.15)
+				)
+				(justify mirror)
+			)
+		)
+		(property "Datasheet" ""
 			(at 0 0 270)
 			(unlocked yes)
@@
 			)
 		)
-		(property "Description" "Generic connector, single row, 01x01, script generated"
+		(property "Description" ""
 			(at 0 0 270)
 			(unlocked yes)
@@
 		(sheetname "/")
 		(sheetfile "non-deployables_XTE-SF.kicad_sch")
-		(attr exclude_from_pos_files)
+		(attr exclude_from_pos_files exclude_from_bom)
 		(fp_rect
 			(start -2.65 5.15)
@@
 		)
 		(fp_text user "${REFERENCE}"
-			(at 0 0 90)
+			(at 0 0 270)
 			(layer "B.Fab")
 			(effects
@@
 	)
 	(segment
-		(start 139.88 62.5)
-		(end 151.13 51.25)
-		(width 2)
-		(layer "F.Cu")
+		(start 50.721 44.399)
+		(end 69.519 44.399)
+		(width 2)
+		(layer "B.Cu")
 		(net 1)
 	)
@@
 		(end 75.12 50)
 		(width 2)
-		(layer "F.Cu")
+		(layer "B.Cu")
 		(net 1)
 	)
 	(segment
-		(start 107.5 62.5)
-		(end 139.88 62.5)
-		(width 2)
-		(layer "F.Cu")
+		(start 144.629 57.751)
+		(end 151.13 51.25)
+		(width 2)
+		(layer "B.Cu")
 		(net 1)
 	)
 	(segment
-		(start 50.721 44.399)
-		(end 69.519 44.399)
-		(width 2)
-		(layer "F.Cu")
+		(start 76.37 51.25)
+		(end 75.12 50)
+		(width 2)
+		(layer "B.Cu")
+		(net 1)
+	)
+	(segment
+		(start 96.25 51.25)
+		(end 76.37 51.25)
+		(width 2)
+		(layer "B.Cu")
+		(net 1)
+	)
+	(segment
+		(start 102.751 57.751)
+		(end 144.629 57.751)
+		(width 2)
+		(layer "B.Cu")
+		(net 1)
+	)
+	(segment
+		(start 96.25 51.25)
+		(end 102.751 57.751)
+		(width 2)
+		(layer "B.Cu")
 		(net 1)
 	)
@@
 		(end 50.721 44.399)
 		(width 2)
-		(layer "F.Cu")
+		(layer "B.Cu")
 		(net 1)
 	)
@@
 	)
 	(segment
+		(start 166.37 51.25)
+		(end 123.75 93.87)
+		(width 2)
+		(layer "B.Cu")
+		(net 3)
+	)
+	(segment
 		(start 123.75 93.87)
 		(end 123.75 118.75)
 		(width 2)
-		(layer "F.Cu")
-		(net 3)
-	)
-	(segment
-		(start 166.37 51.25)
-		(end 123.75 93.87)
-		(width 2)
-		(layer "F.Cu")
+		(layer "B.Cu")
 		(net 3)
 	)
@@
 		(end 31.25 76.25)
 		(width 2)
-		(layer "F.Cu")
+		(layer "B.Cu")
 		(net 4)
 	)
@@
 		(end 29.88 74.88)
 		(width 2)
-		(layer "F.Cu")
+		(layer "B.Cu")
 		(net 4)
 	)
 	(segment
+		(start 222.5 32.38)
+		(end 222.5 92.5)
+		(width 2)
+		(layer "B.Cu")
+		(net 5)
+	)
+	(segment
 		(start 223.63 31.25)
-		(end 222.03 32.85)
-		(width 2)
-		(layer "F.Cu")
+		(end 222.5 32.38)
+		(width 2)
+		(layer "B.Cu")
 		(net 5)
 	)
 	(segment
-		(start 222.03 32.85)
-		(end 222.03 92.03)
-		(width 2)
-		(layer "F.Cu")
+		(start 222.5 92.5)
+		(end 228.75 98.75)
+		(width 2)
+		(layer "B.Cu")
 		(net 5)
 	)
 	(segment
-		(start 222.03 92.03)
-		(end 228.75 98.75)
-		(width 2)
-		(layer "F.Cu")
-		(net 5)
+		(start 396.37 31.25)
+		(end 328.87 98.75)
+		(width 2)
+		(layer "B.Cu")
+		(net 6)
 	)
 	(segment
@@
 		(end 321.25 98.75)
 		(width 2)
-		(layer "F.Cu")
-		(net 6)
-	)
-	(segment
-		(start 396.37 31.25)
-		(end 328.87 98.75)
-		(width 2)
-		(layer "F.Cu")
+		(layer "B.Cu")
 		(net 6)
 	)
@@
 	)
 	(segment
-		(start 247.62 22.5)
-		(end 285 22.5)
-		(width 2)
-		(layer "F.Cu")
+		(start 302.5 22.5)
+		(end 372.38 22.5)
+		(width 2)
+		(layer "B.Cu")
 		(net 14)
 	)
 	(segment
-		(start 373.63 23.75)
-		(end 301.25 23.75)
-		(width 2)
-		(layer "F.Cu")
+		(start 287.249 24.749)
+		(end 293.75 31.25)
+		(width 2)
+		(layer "B.Cu")
 		(net 14)
 	)
 	(segment
+		(start 293.75 31.25)
+		(end 302.5 22.5)
+		(width 2)
+		(layer "B.Cu")
+		(net 14)
+	)
+	(segment
 		(start 238.87 31.25)
-		(end 247.62 22.5)
-		(width 2)
-		(layer "F.Cu")
+		(end 245.371 24.749)
+		(width 2)
+		(layer "B.Cu")
 		(net 14)
 	)
 	(segment
-		(start 285 22.5)
-		(end 293.75 31.25)
-		(width 2)
-		(layer "F.Cu")
+		(start 245.371 24.749)
+		(end 287.249 24.749)
+		(width 2)
+		(layer "B.Cu")
 		(net 14)
 	)
 	(segment
-		(start 301.25 23.75)
-		(end 293.75 31.25)
-		(width 2)
-		(layer "F.Cu")
-		(net 14)
-	)
-	(segment
-		(start 381.13 31.25)
-		(end 373.63 23.75)
-		(width 2)
-		(layer "F.Cu")
+		(start 372.38 22.5)
+		(end 381.13 31.25)
+		(width 2)
+		(layer "B.Cu")
 		(net 14)
 	)
@@
 	(segment
 		(start 193.75 53.75)
-		(end 196.25 51.25)
-		(width 2)
-		(layer "F.Cu")
+		(end 193.75 76.25)
+		(width 2)
+		(layer "B.Cu")
 		(net 20)
 	)
 	(segment
-		(start 193.75 76.25)
+		(start 196.25 51.25)
 		(end 193.75 53.75)
 		(width 2)
-		(layer "F.Cu")
+		(layer "B.Cu")
 		(net 20)
 	)
 	(segment
-		(start 231.25 56.25)
-		(end 256.25 31.25)
-		(width 2)
-		(layer "F.Cu")
+		(start 253.75 31.25)
+		(end 228.75 56.25)
+		(width 2)
+		(layer "B.Cu")
 		(net 21)
 	)
 	(segment
-		(start 228.75 56.25)
-		(end 231.25 56.25)
-		(width 2)
-		(layer "F.Cu")
-		(net 21)
-	)
-	(segment
-		(start 256.25 31.25)
-		(end 266.25 31.25)
-		(width 2)
-		(layer "F.Cu")
+		(start 266.25 31.25)
+		(end 253.75 31.25)
+		(width 2)
+		(layer "B.Cu")
 		(net 21)
 	)
@@
 		(net 23)
 	)
+	(zone
+		(net 25)
+		(net_name "GND2")
+		(layer "B.Cu")
+		(hatch edge 0.5)
+		(priority 1)
+		(connect_pads
+			(clearance 0.5)
+		)
+		(min_thickness 0.25)
+		(filled_areas_thickness no)
+		(fill yes
+			(thermal_gap 0.5)
+			(thermal_bridge_width 0.5)
+		)
+		(polygon
+			(pts
+				(xy 317.5 27.5) (xy 397.5 47.5) (xy 397.5 240) (xy 290 232.5)
+			)
+		)
+	)
+	(zone
+		(net 24)
+		(net_name "GND1")
+		(layer "B.Cu")
+		(hatch edge 0.5)
+		(connect_pads
+			(clearance 0.5)
+		)
+		(min_thickness 0.25)
+		(filled_areas_thickness no)
+		(fill yes
+			(thermal_gap 0.5)
+			(thermal_bridge_width 0.5)
+		)
+		(polygon
+			(pts
+				(xy 117.916667 42.5) (xy 182.286585 42.5) (xy 200 250) (xy 92.857951 265.357951)
+			)
+		)
+	)
 	(embedded_fonts no)

Commit message: updated with mounting holes
Parts:
- added H1: MountingHole_Pad, MountingHole:MountingHole_3.2mm_M3_DIN965_Pad, F.Cu at (25.0, 50.0)
- added H2: MountingHole_Pad, MountingHole:MountingHole_3.2mm_M3_DIN965_Pad, F.Cu at (200.0, 50.0)
- added H3: MountingHole_Pad, MountingHole:MountingHole_3.2mm_M3_DIN965_Pad, F.Cu at (25.0, 272.5)
- added H4: MountingHole_Pad, MountingHole:MountingHole_3.2mm_M3_DIN965_Pad, F.Cu at (200.0, 272.5)
- added H5: MountingHole_Pad, MountingHole:MountingHole_3.2mm_M3_DIN965_Pad, F.Cu at (222.5, 30.0)
- added H6: MountingHole_Pad, MountingHole:MountingHole_3.2mm_M3_DIN965_Pad, F.Cu at (397.5, 30.0)
- added H7: MountingHole_Pad, MountingHole:MountingHole_3.2mm_M3_DIN965_Pad, F.Cu at (222.5, 252.5)
- added H8: MountingHole_Pad, MountingHole:MountingHole_3.2mm_M3_DIN965_Pad, F.Cu at (397.5, 252.5)
- J1, J2: moved to F.Cu
- Other_Board2, gnd_connector1, gnd_connector2: moved to B.Cu
- moved D5 30.0 mm to (351.1, 31.2)
- moved D4 17.1 mm to (256.0, 31.2)
- moved Other_Board1 13.8 mm to (182.5, 51.2)
- moved Other_Board2 11.2 mm to (277.5, 31.2)
- moved D3 5.00 mm to (50.1, 50.0)
Routing:
- net Net-(D4-K): track 154.9 -> 105.9 mm
- net Net-(D5-A): track 103.1 -> 90.7 mm
- net Net-(Other_Board2-Pin_1): track 47.9 -> 59.1 mm
- net Net-(D4-A): track 70.6 -> 77.4 mm
- net Net-(D1-K): track 116.6 -> 111.6 mm
- net Net-(Other_Board1-Pin_1): track 26.0 -> 29.7 mm
- net Net-(D3-A): track 26.8 -> 27.8 mm
Other:
- board size 390 x 252.5 mm -> 387.5 x 260 mm

Commit message: added pcb labels
Parts:
- moved D4 6.37 mm to (257.2, 25.0)
- moved D5 6.37 mm to (352.4, 25.0)
- moved H5 6.37 mm to (223.8, 23.8)
- moved H6 6.37 mm to (398.8, 23.8)
- moved H7 6.37 mm to (223.8, 246.2)
- moved H8 6.37 mm to (398.8, 246.2)
- moved J2 6.37 mm to (295.0, 25.0)
- moved Other_Board2 6.37 mm to (278.8, 25.0)
- moved SC11 6.37 mm to (265.0, 50.0)
- moved SC12 6.37 mm to (357.5, 50.0)
- moved SC13 6.37 mm to (265.0, 92.5)
- moved SC14 6.37 mm to (265.0, 135.0)
- moved SC15 6.37 mm to (265.0, 177.5)
- moved SC16 6.37 mm to (265.0, 220.0)
- moved SC17 6.37 mm to (357.5, 92.5)
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Other:
- board size 387.5 x 260 mm -> 388.8 x 266.2 mm
- board text added: "Protoype Solar Panels 4s5p board 1 University of Washington Husky Satellite Lab HS-2"
- board text added: "Protoype Solar Panels 4s5p board 2 University of Washington Husky Satellite Lab HS-2"
Changed lines of the file:
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@@
 	(footprint "solar_cells:XOLAR_SM401K08TF"
 		(layer "F.Cu")
-		(at 356.25 226.25)
+		(at 357.5 220)
 		(property "Reference" "SC20"
 			(at 0 -0.5 0)
@@
 	(footprint "MountingHole:MountingHole_3.2mm_M3_DIN965_Pad"
 		(layer "F.Cu")
-		(at 397.5 30)
+		(at 398.75 23.75)
 		(descr "Mounting Hole 3.2mm, M3, generated by kicad-footprint-generator mountinghole.py")
 		(tags "mountinghole M3 DIN965")
@@
 	(footprint "solar_cells:XOLAR_SM401K08TF"
 		(layer "F.Cu")
-		(at 356.25 98.75)
+		(at 357.5 92.5)
 		(property "Reference" "SC17"
 			(at 0 -0.5 0)
@@
 	(footprint "MountingHole:MountingHole_3.2mm_M3_DIN965_Pad"
 		(layer "F.Cu")
-		(at 222.5 252.5)
+		(at 223.75 246.25)
 		(descr "Mounting Hole 3.2mm, M3, generated by kicad-footprint-generator mountinghole.py")
 		(tags "mountinghole M3 DIN965")
@@
 	(footprint "solar_cells:XOLAR_SM401K08TF"
 		(layer "F.Cu")
-		(at 356.25 141.25)
+		(at 357.5 135)
 		(property "Reference" "SC18"
 			(at 0 -0.5 0)
@@
 	(footprint "MountingHole:MountingHole_3.2mm_M3_DIN965_Pad"
 		(layer "F.Cu")
-		(at 397.5 252.5)
+		(at 398.75 246.25)
 		(descr "Mounting Hole 3.2mm, M3, generated by kicad-footprint-generator mountinghole.py")
 		(tags "mountinghole M3 DIN965")
@@
 	(footprint "solar_cells:XOLAR_SM401K08TF"
 		(layer "F.Cu")
-		(at 263.75 141.25)
+		(at 265 135)
 		(property "Reference" "SC14"
 			(at 0 -0.5 0)
@@
 	(footprint "Connector_Wire:SolderWirePad_1x01_SMD_5x10mm"
 		(layer "F.Cu")
-		(at 293.75 31.25 90)
+		(at 295 25 90)
 		(descr "Wire Pad, Square, SMD Pad,  5mm x 10mm")
 		(tags "MeasurementPoint Square SMDPad 5mmx10mm ")
@@
 	(footprint "solar_cells:XOLAR_SM401K08TF"
 		(layer "F.Cu")
-		(at 263.75 226.25)
+		(at 265 220)
 		(property "Reference" "SC16"
 			(at 0 -0.5 0)
@@
 	(footprint "solar_cells:XOLAR_SM401K08TF"
 		(layer "F.Cu")
-		(at 356.25 56.25)
+		(at 357.5 50)
 		(property "Reference" "SC12"
 			(at 0 -0.5 0)
@@
 	(footprint "solar_cells:XOLAR_SM401K08TF"
 		(layer "F.Cu")
-		(at 263.75 98.75)
+		(at 265 92.5)
 		(property "Reference" "SC13"
 			(at 0 -0.5 0)
@@
 	(footprint "solar_cells:XOLAR_SM401K08TF"
 		(layer "F.Cu")
-		(at 263.75 183.75)
+		(at 265 177.5)
 		(property "Reference" "SC15"
 			(at 0 -0.5 0)
@@
 	(footprint "MountingHole:MountingHole_3.2mm_M3_DIN965_Pad"
 		(layer "F.Cu")
-		(at 222.5 30)
+		(at 223.75 23.75)
 		(descr "Mounting Hole 3.2mm, M3, generated by kicad-footprint-generator mountinghole.py")
 		(tags "mountinghole M3 DIN965")
@@
 	(footprint "solar_cells:XOLAR_SM401K08TF"
 		(layer "F.Cu")
-		(at 356.25 183.75)
+		(at 357.5 177.5)
 		(property "Reference" "SC19"
 			(at 0 -0.5 0)
@@
 	(footprint "solar_cells:XOLAR_SM401K08TF"
 		(layer "F.Cu")
-		(at 263.75 56.25)
+		(at 265 50)
 		(property "Reference" "SC11"
 			(at 0 -0.5 0)
@@
 	(footprint "Diode_THT:D_DO-201AD_P15.24mm_Horizontal"
 		(layer "B.Cu")
-		(at 256 31.25 180)
+		(at 257.25 25 180)
 		(descr "Diode, DO-201AD series, Axial, Horizontal, pin pitch=15.24mm, length*diameter=9.5*5.2mm^2, http://www.diodes.com/_files/packages/DO-201AD.pdf")
 		(tags "Diode DO-201AD series Axial Horizontal pin pitch 15.24mm  length 9.5mm diameter 5.2mm")
@@
 	(footprint "Diode_THT:D_DO-201AD_P15.24mm_Horizontal"
 		(layer "B.Cu")
-		(at 351.13 31.25)
+		(at 352.38 25)
 		(descr "Diode, DO-201AD series, Axial, Horizontal, pin pitch=15.24mm, length*diameter=9.5*5.2mm^2, http://www.diodes.com/_files/packages/DO-201AD.pdf")
 		(tags "Diode DO-201AD series Axial Horizontal pin pitch 15.24mm  length 9.5mm diameter 5.2mm")
@@
 	(footprint "Connector_Wire:SolderWirePad_1x01_SMD_5x10mm"
 		(layer "B.Cu")
-		(at 277.5 31.25 90)
+		(at 278.75 25 90)
 		(descr "Wire Pad, Square, SMD Pad,  5mm x 10mm")
 		(tags "MeasurementPoint Square SMDPad 5mmx10mm ")
@@
 	(footprint "Connector_Wire:SolderWirePad_1x01_SMD_5x10mm"
 		(layer "B.Cu")
-		(at 326.25 31.25 90)
+		(at 327.5 25 90)
 		(descr "Wire Pad, Square, SMD Pad,  5mm x 10mm")
 		(tags "MeasurementPoint Square SMDPad 5mmx10mm ")
@@
 	)
 	(gr_rect
-		(start 215 20)
-		(end 405 260)
+		(start 216.25 13.75)
+		(end 406.25 253.75)
 		(stroke
 			(width 0.05)
@@
 		(layer "Edge.Cuts")
 	)
+	(gr_text "Protoype Solar Panels 4s5p board 2\nUniversity of Washington\nHusky Satellite Lab HS-2\n"
+		(at 313.75 251.25 0)
+		(layer "F.SilkS")
+		(effects
+			(font
+				(size 2 2)
+				(thickness 0.25)
+			)
+			(justify bottom)
+		)
+	)
+	(gr_text "Protoype Solar Panels 4s5p board 1\nUniversity of Washington\nHusky Satellite Lab HS-2\n"
+		(at 110 277.5 0)
+		(layer "F.SilkS")
+		(effects
+			(font
+				(size 2 2)
+				(thickness 0.25)
+			)
+			(justify bottom)
+		)
+	)
 	(segment
 		(start 102.751 57.751)
@@
 	)
 	(segment
-		(start 222.749 49.261)
-		(end 222.749 92.749)
+		(start 223.999 43.011)
+		(end 223.999 86.499)
 		(width 2)
 		(layer "B.Cu")
@@
 	)
 	(segment
-		(start 222.749 92.749)
-		(end 228.75 98.75)
+		(start 223.999 86.499)
+		(end 230 92.5)
 		(width 2)
 		(layer "B.Cu")
@@
 	)
 	(segment
-		(start 240.76 31.25)
-		(end 222.749 49.261)
+		(start 242.01 25)
+		(end 223.999 43.011)
 		(width 2)
 		(layer "B.Cu")
@@
 	)
 	(segment
-		(start 328.87 98.75)
-		(end 328.87 68.75)
+		(start 330.12 92.5)
+		(end 330.12 62.5)
 		(width 2)
 		(layer "B.Cu")
@@
 	)
 	(segment
-		(start 328.87 68.75)
-		(end 366.37 31.25)
+		(start 330.12 62.5)
+		(end 367.62 25)
 		(width 2)
 		(layer "B.Cu")
@@
 	)
 	(segment
-		(start 328.87 98.75)
-		(end 321.25 98.75)
+		(start 330.12 92.5)
+		(end 322.5 92.5)
 		(width 2)
 		(layer "B.Cu")
@@
 	)
 	(segment
-		(start 300.251 24.749)
-		(end 344.629 24.749)
+		(start 301.501 18.499)
+		(end 345.879 18.499)
 		(width 2)
 		(layer "B.Cu")
@@
 	)
 	(segment
-		(start 344.629 24.749)
-		(end 351.13 31.25)
+		(start 345.879 18.499)
+		(end 352.38 25)
 		(width 2)
 		(layer "B.Cu")
@@
 	)
 	(segment
-		(start 256 31.25)
-		(end 262.501 24.749)
+		(start 257.25 25)
+		(end 263.751 18.499)
 		(width 2)
 		(layer "B.Cu")
@@
 	)
 	(segment
-		(start 287.249 24.749)
-		(end 293.75 31.25)
+		(start 288.499 18.499)
+		(end 295 25)
 		(width 2)
 		(layer "B.Cu")
@@
 	)
 	(segment
-		(start 293.75 31.25)
-		(end 300.251 24.749)
+		(start 295 25)
+		(end 301.501 18.499)
 		(width 2)
 		(layer "B.Cu")
@@
 	)
 	(segment
-		(start 262.501 24.749)
-		(end 287.249 24.749)
+		(start 263.751 18.499)
+		(end 288.499 18.499)
 		(width 2)
 		(layer "B.Cu")
@@
 	)
 	(segment
-		(start 271.25 98.75)
-		(end 298.75 98.75)
+		(start 272.5 92.5)
+		(end 300 92.5)
 		(width 2)
 		(layer "F.Cu")
@@
 	)
 	(segment
-		(start 228.75 141.25)
-		(end 271.25 98.75)
+		(start 230 135)
+		(end 272.5 92.5)
 		(width 2)
 		(layer "F.Cu")
@@
 	)
 	(segment
-		(start 228.75 183.75)
-		(end 271.25 141.25)
+		(start 230 177.5)
+		(end 272.5 135)
 		(width 2)
 		(layer "F.Cu")
@@
 	)
 	(segment
-		(start 271.25 141.25)
-		(end 298.75 141.25)
+		(start 272.5 135)
+		(end 300 135)
 		(width 2)
 		(layer "F.Cu")
@@
 	)
 	(segment
-		(start 298.75 183.75)
-		(end 271.25 183.75)
+		(start 300 177.5)
+		(end 272.5 177.5)
 		(width 2)
 		(layer "F.Cu")
@@
 	)
 	(segment
-		(start 271.25 183.75)
-		(end 228.75 226.25)
+		(start 272.5 177.5)
+		(end 230 220)
 		(width 2)
 		(layer "F.Cu")
@@
 	)
 	(segment
-		(start 363.75 98.75)
-		(end 321.25 141.25)
+		(start 365 92.5)
+		(end 322.5 135)
 		(width 2)
 		(layer "F.Cu")
@@
 	)
 	(segment
-		(start 391.25 98.75)
-		(end 363.75 98.75)
+		(start 392.5 92.5)
+		(end 365 92.5)
 		(width 2)
 		(layer "F.Cu")
@@
 	)
 	(segment
-		(start 363.75 141.25)
-		(end 321.25 183.75)
+		(start 365 135)
+		(end 322.5 177.5)
 		(width 2)
 		(layer "F.Cu")
@@
 	)
 	(segment
-		(start 391.25 141.25)
-		(end 363.75 141.25)
+		(start 392.5 135)
+		(end 365 135)
 		(width 2)
 		(layer "F.Cu")
@@
 	)
 	(segment
-		(start 228.75 56.25)
-		(end 252.5 56.25)
+		(start 230 50)
+		(end 253.75 50)
 		(width 2)
 		(layer "B.Cu")
@@
 	)
 	(segment
-		(start 252.5 56.25)
-		(end 277.5 31.25)
+		(start 253.75 50)
+		(end 278.75 25)
 		(width 2)
 		(layer "B.Cu")
@@
 	)
 	(segment
-		(start 391.25 183.75)
-		(end 363.75 183.75)
+		(start 392.5 177.5)
+		(end 365 177.5)
 		(width 2)
 		(layer "F.Cu")
@@
 	)
 	(segment
-		(start 363.75 183.75)
-		(end 321.25 226.25)
+		(start 365 177.5)
+		(end 322.5 220)
 		(width 2)
 		(layer "F.Cu")
@@
 	)
 	(segment
-		(start 298.75 56.25)
-		(end 321.25 56.25)
+		(start 300 50)
+		(end 322.5 50)
 		(width 2)
 		(layer "F.Cu")
@@
 		(polygon
 			(pts
-				(xy 217.5 25) (xy 402.5 25) (xy 402.5 257.5) (xy 217.5 257.5)
+				(xy 218.75 18.75) (xy 403.75 18.75) (xy 403.75 251.25) (xy 218.75 251.25)
 			)
 		)
