File: hs2/non-deployables-XTE-SF/non-deployables-XTE-SF.kicad_sch (KiCad schematic)
At the start: 9 parts, among them J1 Conn_01x01_Pin

Commit message: ver 1.0 of xte-sf board
Parts:
- added GND_J1: Conn_01x01_Pin, Connector_Wire:SolderWirePad_1x01_SMD_5x10mm, symbol Connector:Conn_01x01_Pin
Connections:
- net GND: now also GND_J1.1 (Pin_1)
Changed lines of the file:
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@@
+	(wire
+		(pts
+			(xy 38.1 38.1) (xy 38.1 44.45)
+		)
+		(stroke
+			(width 0)
+			(type default)
+		)
+	)
 	(wire
 		(pts
@@
 	(wire
 		(pts
-			(xy 49.53 46.99) (xy 49.53 53.34)
+			(xy 25.4 38.1) (xy 25.4 44.45)
 		)
 		(stroke
@@
 	(symbol
 		(lib_id "power:GND")
-		(at 49.53 53.34 0)
+		(at 25.4 44.45 0)
 		(unit 1)
 		(exclude_from_sim no)
@@
 		(fields_autoplaced yes)
 		(property "Reference" "#PWR01"
-			(at 49.53 59.69 0)
+			(at 25.4 50.8 0)
 			(effects
 				(font
@@
 		)
 		(property "Value" "GND"
-			(at 49.53 58.42 0)
+			(at 25.4 49.53 0)
 			(effects
 				(font
@@
 		)
 		(property "Footprint" ""
-			(at 49.53 53.34 0)
+			(at 25.4 44.45 0)
 			(effects
 				(font
@@
 		)
 		(property "Datasheet" ""
-			(at 49.53 53.34 0)
+			(at 25.4 44.45 0)
 			(effects
 				(font
@@
 		)
 		(property "Description" "Power symbol creates a global label with name \"GND\" , ground"
-			(at 49.53 53.34 0)
+			(at 25.4 44.45 0)
 			(effects
 				(font
@@
 				(path "/dbc43d45-a017-4e42-aa9f-af2b8f794c11"
 					(reference "#PWR01")
+					(unit 1)
+				)
+			)
+		)
+	)
+	(symbol
+		(lib_id "power:GND")
+		(at 38.1 44.45 0)
+		(unit 1)
+		(exclude_from_sim no)
+		(in_bom yes)
+		(on_board yes)
+		(dnp no)
+		(fields_autoplaced yes)
+		(property "Reference" "#PWR03"
+			(at 38.1 50.8 0)
+			(effects
+				(font
+					(size 1.27 1.27)
+				)
+				(hide yes)
+			)
+		)
+		(property "Value" "GND"
+			(at 38.1 49.53 0)
+			(effects
+				(font
+					(size 1.27 1.27)
+				)
+			)
+		)
+		(property "Footprint" ""
+			(at 38.1 44.45 0)
+			(effects
+				(font
+					(size 1.27 1.27)
+				)
+				(hide yes)
+			)
+		)
+		(property "Datasheet" ""
+			(at 38.1 44.45 0)
+			(effects
+				(font
+					(size 1.27 1.27)
+				)
+				(hide yes)
+			)
+		)
+		(property "Description" "Power symbol creates a global label with name \"GND\" , ground"
+			(at 38.1 44.45 0)
+			(effects
+				(font
+					(size 1.27 1.27)
+				)
+				(hide yes)
+			)
+		)
+		(pin "1"
+		)
+		(instances
+			(project "spectrolab_4x7_design"
+				(path "/dbc43d45-a017-4e42-aa9f-af2b8f794c11"
+					(reference "#PWR03")
 					(unit 1)
 				)
@@
 	)
 	(symbol
+		(lib_id "Connector:Conn_01x01_Pin")
+		(at 38.1 33.02 270)
+		(unit 1)
+		(exclude_from_sim no)
+		(in_bom yes)
+		(on_board yes)
+		(dnp no)
+		(fields_autoplaced yes)
+		(property "Reference" "GND_J1"
+			(at 39.37 32.3849 90)
+			(effects
+				(font
+					(size 1.27 1.27)
+				)
+				(justify left)
+			)
+		)
+		(property "Value" "Conn_01x01_Pin"
+			(at 39.37 34.9249 90)
+			(effects
+				(font
+					(size 1.27 1.27)
+				)
+				(justify left)
+			)
+		)
+		(property "Footprint" "Connector_Wire:SolderWirePad_1x01_SMD_5x10mm"
+			(at 38.1 33.02 0)
+			(effects
+				(font
+					(size 1.27 1.27)
+				)
+				(hide yes)
+			)
+		)
+		(property "Datasheet" "~"
+			(at 38.1 33.02 0)
+			(effects
+				(font
+					(size 1.27 1.27)
+				)
+				(hide yes)
+			)
+		)
+		(property "Description" "Generic connector, single row, 01x01, script generated"
+			(at 38.1 33.02 0)
+			(effects
+				(font
+					(size 1.27 1.27)
+				)
+				(hide yes)
+			)
+		)
+		(pin "1"
+		)
+		(instances
+			(project "spectrolab_4x7_design"
+				(path "/dbc43d45-a017-4e42-aa9f-af2b8f794c11"
+					(reference "GND_J1")
+					(unit 1)
+				)
+			)
+		)
+	)
+	(symbol
 		(lib_id "Device:XTE-SF")
 		(at 125.73 55.88 90)
@@
 	(symbol
 		(lib_id "power:PWR_FLAG")
-		(at 49.53 46.99 0)
+		(at 25.4 38.1 0)
 		(unit 1)
 		(exclude_from_sim no)
@@
 		(fields_autoplaced yes)
 		(property "Reference" "#FLG01"
-			(at 49.53 45.085 0)
+			(at 25.4 36.195 0)
 			(effects
 				(font
@@
 		)
 		(property "Value" "PWR_FLAG"
-			(at 49.53 41.91 0)
+			(at 25.4 33.02 0)
 			(effects
 				(font
@@
 		)
 		(property "Footprint" ""
-			(at 49.53 46.99 0)
+			(at 25.4 38.1 0)
 			(effects
 				(font
@@
 		)
 		(property "Datasheet" "~"
-			(at 49.53 46.99 0)
+			(at 25.4 38.1 0)
 			(effects
 				(font
@@
 		)
 		(property "Description" "Special symbol for telling ERC where power comes from"
-			(at 49.53 46.99 0)
-			(effects
-				(font
+			(at 25.4 38.1 0)
+			(effects
+				(font

Commit message: started stack KiCAD
Connections:
- net GND: no longer GND_J1.1 (Pin_1)
- new net BMS: GND_J1.1 (Pin_1)
Other:
- moved on the sheet: GND_J1
Changed lines of the file:
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@@
-	(wire
-		(pts
-			(xy 38.1 38.1) (xy 38.1 44.45)
-		)
-		(stroke
-			(width 0)
-			(type default)
-		)
-	)
 	(wire
 		(pts
@@
 			(width 0)
 			(type default)
+		)
+	)
+	(global_label "BMS"
+		(shape output)
+		(at 48.26 43.18 90)
+		(fields_autoplaced yes)
+		(effects
+			(font
+				(size 1.27 1.27)
+			)
+			(justify left)
+		)
+		(property "Intersheetrefs" "${INTERSHEET_REFS}"
+			(at 48.26 36.2639 90)
+			(effects
+				(font
+					(size 1.27 1.27)
+				)
+				(justify left)
+				(hide yes)
+			)
 		)
 	)
@@
 	)
 	(symbol
-		(lib_id "power:GND")
-		(at 38.1 44.45 0)
-		(unit 1)
-		(exclude_from_sim no)
-		(in_bom yes)
-		(on_board yes)
-		(dnp no)
-		(fields_autoplaced yes)
-		(property "Reference" "#PWR03"
-			(at 38.1 50.8 0)
-			(effects
-				(font
-					(size 1.27 1.27)
-				)
-				(hide yes)
-			)
-		)
-		(property "Value" "GND"
-			(at 38.1 49.53 0)
-			(effects
-				(font
-					(size 1.27 1.27)
-				)
-			)
-		)
-		(property "Footprint" ""
-			(at 38.1 44.45 0)
-			(effects
-				(font
-					(size 1.27 1.27)
-				)
-				(hide yes)
-			)
-		)
-		(property "Datasheet" ""
-			(at 38.1 44.45 0)
-			(effects
-				(font
-					(size 1.27 1.27)
-				)
-				(hide yes)
-			)
-		)
-		(property "Description" "Power symbol creates a global label with name \"GND\" , ground"
-			(at 38.1 44.45 0)
-			(effects
-				(font
-					(size 1.27 1.27)
-				)
-				(hide yes)
-			)
-		)
-		(pin "1"
-		)
-		(instances
-			(project "spectrolab_4x7_design"
-				(path "/dbc43d45-a017-4e42-aa9f-af2b8f794c11"
-					(reference "#PWR03")
-					(unit 1)
-				)
-			)
-		)
-	)
-	(symbol
 		(lib_id "Device:XTE-SF")
 		(at 151.13 55.88 90)
@@
 	(symbol
 		(lib_id "Connector:Conn_01x01_Pin")
-		(at 38.1 33.02 270)
-		(unit 1)
-		(exclude_from_sim no)
-		(in_bom yes)
-		(on_board yes)
-		(dnp no)
-		(fields_autoplaced yes)
+		(at 48.26 48.26 90)
+		(unit 1)
+		(exclude_from_sim no)
+		(in_bom yes)
+		(on_board yes)
+		(dnp no)
 		(property "Reference" "GND_J1"
-			(at 39.37 32.3849 90)
+			(at 46.99 48.8951 90)
 			(effects
 				(font
@@
 		)
 		(property "Value" "Conn_01x01_Pin"
-			(at 39.37 34.9249 90)
+			(at 46.99 46.3551 90)
 			(effects
 				(font
@@
 		)
 		(property "Footprint" "Connector_Wire:SolderWirePad_1x01_SMD_5x10mm"
-			(at 38.1 33.02 0)
+			(at 48.26 48.26 0)
 			(effects
 				(font
@@
 		)
 		(property "Datasheet" "~"
-			(at 38.1 33.02 0)
+			(at 48.26 48.26 0)
 			(effects
 				(font
@@
 		)
 		(property "Description" "Generic connector, single row, 01x01, script generated"
-			(at 38.1 33.02 0)
-			(effects
-				(font
+			(at 48.26 48.26 0)
+			(effects
+				(font
